Commit message: added slam

File: description/robot.urdf.xacro (robot description, xacro)
@@ -2,4 +2,5 @@
 <robot xmlns:xacro="http://www.ros.org/wiki/xacro"  name="robot">
     <xacro:arg name="use_ros2_control" default='true'/>
+    <xacro:arg name="sim_mode" default='false'/>
     <xacro:include filename='constants.xacro'/>
     <xacro:include filename="robot_core.xacro"/>

File: description/robot_core.xacro (robot description, xacro)
@@ -4,4 +4,12 @@
     <!-- Base Link -->
     <link name="base_link">
+    </link>
+    <!-- Chassis -->
+    <joint name="base_footprint_joint" type="fixed">
+        <parent link="base_link"/>
+        <child link="base_footprint"/>
+        <origin xyz="0 0 0" rpy="0 0 0"/>
+    </joint>
+    <link name="base_footprint">
     </link>
     <!-- Chassis -->

File: description/ros2_control.xacro (robot description, xacro)
@@ -1,58 +1,62 @@
 <?xml version="1.0"?>
 <robot xmlns:xacro="http://www.ros.org/wiki/xacro">
-    <ros2_control name="RealSys" type="system">
-        <hardware>
-            <plugin>diffdrive_arduino/DiffDriveArduino</plugin>
-            <param name="left_wheel_name">left_wheel_joint</param>
-            <param name="right_wheel_name">right_wheel_joint</param>
-            <param name="loop_rate">${pid_loop_rate}</param>
-            <param name="device">/dev/ttyUSB0</param>
-            <param name="baud_rate">57600</param>
-            <param name="timeout">1000</param>
-            <param name="enc_count_per_rev">${enc_count_per_rev}</param>
-        </hardware>
-        <joint name="left_wheel_joint">
-            <command_interface name="velocity">
-                <param name='min'>-10</param>
-                <param name='max'>10</param>
-            </command_interface>
-            <state_interface name="velocity"/>
-            <state_interface name="position"/>
-        </joint>
-        <joint name="right_wheel_joint">
-            <command_interface name="velocity">
-                <param name='min'>-10</param>
-                <param name='max'>10</param>
-            </command_interface>
-            <state_interface name="velocity"/>
-            <state_interface name="position"/>
-        </joint>
-    </ros2_control>
-    <!-- this plugin will tell ros how to talk to gazrbo -->
-    <!-- <ros2_control name="GazSys" type="system">
-        <hardware>
-            <plugin>gazebo_ros2_control/GazeboSystem</plugin>
-        </hardware>
-        <joint name="left_wheel_joint">
-            <command_interface name="velocity">
-                <param name='min'>-10</param>
-                <param name='max'>10</param>
-            </command_interface>
-            <state_interface name="velocity"/>
-            <state_interface name="position"/>
-        </joint>
-        <joint name="right_wheel_joint">
-            <command_interface name="velocity">
-                <param name='min'>-10</param>
-                <param name='max'>10</param>
-            </command_interface>
-            <state_interface name="velocity"/>
-            <state_interface name="position"/>
-        </joint>
-    </ros2_control> -->
-    <gazebo>
-        <plugin name="gazebo_ros2_cont" filename="libgazebo_ros2_control.so">
-            <parameters>$(find my_bot2)/config/my_controllers.yaml</parameters>
-        </plugin>
-    </gazebo>
+    <xacro:unless value="$(arg sim_mode)">
+        <ros2_control name="RealSys" type="system">
+            <hardware>
+                <plugin>diffdrive_arduino/DiffDriveArduino</plugin>
+                <param name="left_wheel_name">left_wheel_joint</param>
+                <param name="right_wheel_name">right_wheel_joint</param>
+                <param name="loop_rate">${pid_loop_rate}</param>
+                <param name="device">/dev/ttyUSB0</param>
+                <param name="baud_rate">57600</param>
+                <param name="timeout">1000</param>
+                <param name="enc_count_per_rev">${enc_count_per_rev}</param>
+            </hardware>
+            <joint name="left_wheel_joint">
+                <command_interface name="velocity">
+                    <param name='min'>-10</param>
+                    <param name='max'>10</param>
+                </command_interface>
+                <state_interface name="velocity"/>
+                <state_interface name="position"/>
+            </joint>
+            <joint name="right_wheel_joint">
+                <command_interface name="velocity">
+                    <param name='min'>-10</param>
+                    <param name='max'>10</param>
+                </command_interface>
+                <state_interface name="velocity"/>
+                <state_interface name="position"/>
+            </joint>
+        </ros2_control>
+    </xacro:unless>
+    <xacro:if value="$(arg sim_mode)">
+        <ros2_control name="GazSys" type="system">
+            <hardware>
+                <!-- this plugin will tell ros how to talk to gazrbo -->
+                <plugin>gazebo_ros2_control/GazeboSystem</plugin>
+            </hardware>
+            <joint name="left_wheel_joint">
+                <command_interface name="velocity">
+                    <param name='min'>-10</param>
+                    <param name='max'>10</param>
+                </command_interface>
+                <state_interface name="velocity"/>
+                <state_interface name="position"/>
+            </joint>
+            <joint name="right_wheel_joint">
+                <command_interface name="velocity">
+                    <param name='min'>-10</param>
+                    <param name='max'>10</param>
+                </command_interface>
+                <state_interface name="velocity"/>
+                <state_interface name="position"/>
+            </joint>
+        </ros2_control>
+        <gazebo>
+            <plugin name="gazebo_ros2_cont" filename="libgazebo_ros2_control.so">
+                <parameters>$(find my_bot2)/config/my_controllers.yaml</parameters>
+            </plugin>
+        </gazebo>
+    </xacro:if>
 </robot>
