Commit message: added real robot controller manager NOT TESTED YET

File: description/constants.xacro (robot description, xacro)
@@ -2,12 +2,15 @@
 <robot xmlns:xacro="http://www.ros.org/wiki/xacro">
     <!-- Constants -->
+    <!-- chassis -->
     <xacro:property name='chss_len' value='0.8'/>
     <xacro:property name='chss_wid' value='0.8'/>
     <xacro:property name='chss_h' value='0.325'/>
     <xacro:property name='chss_mass' value='5'/>
+    <!-- wheel -->
     <xacro:property name='wheel_to_origin' value='0.27'/>
     <xacro:property name='wheel_rad' value='0.1'/>
     <xacro:property name='wheel_wid' value='0.02'/>
     <xacro:property name='wheel_mass' value='0.25'/>
+    <!-- caster wheel -->
     <xacro:property name='caster_rad' value='0.1'/>
     <xacro:property name='caster_mass' value='0.2'/>
@@ -15,7 +18,11 @@
     <xacro:property name='back_caster_to_x' value='0.25'/>
     <xacro:property name='back_caster_to_y' value='0.25'/>
+    <!-- lidar -->
     <xacro:property name='lidar_rad' value='0.035'/>
     <xacro:property name='lidar_h' value='0.054'/>
     <xacro:property name='lidar_h_to_cam' value='0.044'/>
+    <!-- controller -->
+    <xacro:property name='pid_loop_rate' value='30'/>
+    <xacro:property name='enc_count_per_rev' value='300'/>
     <!-- Creating colors -->
     <material name="white">

File: description/ros2_control.xacro (robot description, xacro)
@@ -1,6 +1,35 @@
 <?xml version="1.0"?>
 <robot xmlns:xacro="http://www.ros.org/wiki/xacro">
-    <ros2_control name="GazSys" type="system">
-        <hardware> <!-- this plugin will tell ros how to talk to gazrbo-->
+    <ros2_control name="RealSys" type="system">
+        <hardware>
+            <plugin>diffdrive_arduino/DiffDriveArduino</plugin>
+            <param name="left_wheel_name">left_wheel_joint</param>
+            <param name="right_wheel_name">right_wheel_joint</param>
+            <param name="loop_rate">${pid_loop_rate}</param>
+            <param name="device">/dev/ttyUSB0</param>
+            <param name="baud_rate">57600</param>
+            <param name="timeout">1000</param>
+            <param name="enc_count_per_rev">${enc_count_per_rev}</param>
+        </hardware>
+        <joint name="left_wheel_joint">
+            <command_interface name="velocity">
+                <param name='min'>-10</param>
+                <param name='max'>10</param>
+            </command_interface>
+            <state_interface name="velocity"/>
+            <state_interface name="position"/>
+        </joint>
+        <joint name="right_wheel_joint">
+            <command_interface name="velocity">
+                <param name='min'>-10</param>
+                <param name='max'>10</param>
+            </command_interface>
+            <state_interface name="velocity"/>
+            <state_interface name="position"/>
+        </joint>
+    </ros2_control>
+    <!-- this plugin will tell ros how to talk to gazrbo -->
+    <!-- <ros2_control name="GazSys" type="system">
+        <hardware>
             <plugin>gazebo_ros2_control/GazeboSystem</plugin>
         </hardware>
@@ -21,5 +50,5 @@
             <state_interface name="position"/>
         </joint>
-    </ros2_control>
+    </ros2_control> -->
     <gazebo>
         <plugin name="gazebo_ros2_cont" filename="libgazebo_ros2_control.so">

Commit message: edit the robot dimensions

File: description/constants.xacro (robot description, xacro)
@@ -3,19 +3,32 @@
     <!-- Constants -->
     <!-- chassis -->
-    <xacro:property name='chss_len' value='0.8'/>
+    <!-- <xacro:property name='chss_len' value='0.8'/>
     <xacro:property name='chss_wid' value='0.8'/>
     <xacro:property name='chss_h' value='0.325'/>
-    <xacro:property name='chss_mass' value='5'/>
+    <xacro:property name='chss_mass' value='5'/> -->
+    <xacro:property name='chss_len' value='0.26'/>
+    <xacro:property name='chss_wid' value='0.16'/>
+    <xacro:property name='chss_h' value='0.8'/>
+    <xacro:property name='chss_mass' value='2'/>
     <!-- wheel -->
-    <xacro:property name='wheel_to_origin' value='0.27'/>
+    <!-- <xacro:property name='wheel_to_origin' value='0.27'/>
     <xacro:property name='wheel_rad' value='0.1'/>
     <xacro:property name='wheel_wid' value='0.02'/>
-    <xacro:property name='wheel_mass' value='0.25'/>
+    <xacro:property name='wheel_mass' value='0.25'/> -->
+    <xacro:property name='wheel_to_origin' value='0.07'/>
+    <xacro:property name='wheel_rad' value='0.035'/>
+    <xacro:property name='wheel_wid' value='0.02'/>
+    <xacro:property name='wheel_mass' value='0.05'/>
     <!-- caster wheel -->
-    <xacro:property name='caster_rad' value='0.1'/>
+    <!-- <xacro:property name='caster_rad' value='0.1'/>
     <xacro:property name='caster_mass' value='0.2'/>
     <xacro:property name='front_caster_to_origin' value='0.25'/>
     <xacro:property name='back_caster_to_x' value='0.25'/>
-    <xacro:property name='back_caster_to_y' value='0.25'/>
+    <xacro:property name='back_caster_to_y' value='0.25'/> -->
+    <xacro:property name='caster_rad' value='0.035'/>
+    <xacro:property name='caster_mass' value='0.02'/>
+    <xacro:property name='front_caster_to_origin' value='0.1'/>
+    <xacro:property name='back_caster_to_x' value='0.8'/>
+    <xacro:property name='back_caster_to_y' value='0.6'/>
     <!-- lidar -->
     <xacro:property name='lidar_rad' value='0.035'/>

Commit message: edit the robot dimensions

File: description/constants.xacro (robot description, xacro)
@@ -29,6 +29,6 @@
     <xacro:property name='caster_mass' value='0.02'/>
     <xacro:property name='front_caster_to_origin' value='0.1'/>
-    <xacro:property name='back_caster_to_x' value='0.8'/>
-    <xacro:property name='back_caster_to_y' value='0.6'/>
+    <xacro:property name='back_caster_to_x' value='0.08'/>
+    <xacro:property name='back_caster_to_y' value='0.06'/>
     <!-- lidar -->
     <xacro:property name='lidar_rad' value='0.035'/>

Commit message: added launch files

File: description/constants.xacro (robot description, xacro)
@@ -3,32 +3,32 @@
     <!-- Constants -->
     <!-- chassis -->
-    <!-- <xacro:property name='chss_len' value='0.8'/>
+    <xacro:property name='chss_len' value='0.8'/>
     <xacro:property name='chss_wid' value='0.8'/>
     <xacro:property name='chss_h' value='0.325'/>
-    <xacro:property name='chss_mass' value='5'/> -->
-    <xacro:property name='chss_len' value='0.26'/>
+    <xacro:property name='chss_mass' value='5'/>
+    <!-- <xacro:property name='chss_len' value='0.26'/>
     <xacro:property name='chss_wid' value='0.16'/>
     <xacro:property name='chss_h' value='0.8'/>
-    <xacro:property name='chss_mass' value='2'/>
+    <xacro:property name='chss_mass' value='2'/> -->
     <!-- wheel -->
-    <!-- <xacro:property name='wheel_to_origin' value='0.27'/>
+    <xacro:property name='wheel_to_origin' value='0.27'/>
     <xacro:property name='wheel_rad' value='0.1'/>
     <xacro:property name='wheel_wid' value='0.02'/>
-    <xacro:property name='wheel_mass' value='0.25'/> -->
-    <xacro:property name='wheel_to_origin' value='0.07'/>
+    <xacro:property name='wheel_mass' value='0.25'/>
+    <!-- <xacro:property name='wheel_to_origin' value='0.07'/>
     <xacro:property name='wheel_rad' value='0.035'/>
     <xacro:property name='wheel_wid' value='0.02'/>
-    <xacro:property name='wheel_mass' value='0.05'/>
+    <xacro:property name='wheel_mass' value='0.05'/> -->
     <!-- caster wheel -->
-    <!-- <xacro:property name='caster_rad' value='0.1'/>
+    <xacro:property name='caster_rad' value='0.1'/>
     <xacro:property name='caster_mass' value='0.2'/>
     <xacro:property name='front_caster_to_origin' value='0.25'/>
     <xacro:property name='back_caster_to_x' value='0.25'/>
-    <xacro:property name='back_caster_to_y' value='0.25'/> -->
-    <xacro:property name='caster_rad' value='0.035'/>
+    <xacro:property name='back_caster_to_y' value='0.25'/>
+    <!-- <xacro:property name='caster_rad' value='0.035'/>
     <xacro:property name='caster_mass' value='0.02'/>
     <xacro:property name='front_caster_to_origin' value='0.1'/>
     <xacro:property name='back_caster_to_x' value='0.08'/>
-    <xacro:property name='back_caster_to_y' value='0.06'/>
+    <xacro:property name='back_caster_to_y' value='0.06'/> -->
     <!-- lidar -->
     <xacro:property name='lidar_rad' value='0.035'/>

Commit message: a

File: description/constants.xacro (robot description, xacro)
@@ -12,5 +12,5 @@
     <xacro:property name='chss_mass' value='2'/> -->
     <!-- wheel -->
-    <xacro:property name='wheel_to_origin' value='0.27'/>
+    <xacro:property name='wheel_to_origin' value='0.275'/>
     <xacro:property name='wheel_rad' value='0.1'/>
     <xacro:property name='wheel_wid' value='0.02'/>

Commit message: difference between real and mejds robot

File: description/constants.xacro (robot description, xacro)
@@ -2,33 +2,32 @@
 <robot xmlns:xacro="http://www.ros.org/wiki/xacro">
     <!-- Constants -->
-    <!-- chassis -->
-    <xacro:property name='chss_len' value='0.8'/>
+    <!-- REAL ROBOT -->
+    <!-- <xacro:property name='chss_len' value='0.8'/>
     <xacro:property name='chss_wid' value='0.8'/>
     <xacro:property name='chss_h' value='0.325'/>
     <xacro:property name='chss_mass' value='5'/>
-    <!-- <xacro:property name='chss_len' value='0.26'/>
-    <xacro:property name='chss_wid' value='0.16'/>
-    <xacro:property name='chss_h' value='0.8'/>
-    <xacro:property name='chss_mass' value='2'/> -->
-    <!-- wheel -->
     <xacro:property name='wheel_to_origin' value='0.275'/>
     <xacro:property name='wheel_rad' value='0.1'/>
     <xacro:property name='wheel_wid' value='0.02'/>
     <xacro:property name='wheel_mass' value='0.25'/>
-    <!-- <xacro:property name='wheel_to_origin' value='0.07'/>
-    <xacro:property name='wheel_rad' value='0.035'/>
-    <xacro:property name='wheel_wid' value='0.02'/>
-    <xacro:property name='wheel_mass' value='0.05'/> -->
-    <!-- caster wheel -->
     <xacro:property name='caster_rad' value='0.1'/>
     <xacro:property name='caster_mass' value='0.2'/>
     <xacro:property name='front_caster_to_origin' value='0.25'/>
     <xacro:property name='back_caster_to_x' value='0.25'/>
-    <xacro:property name='back_caster_to_y' value='0.25'/>
-    <!-- <xacro:property name='caster_rad' value='0.035'/>
+    <xacro:property name='back_caster_to_y' value='0.25'/> -->
+    <!-- MEJD'S ROBOT -->
+    <xacro:property name='chss_len' value='0.26'/>
+    <xacro:property name='chss_wid' value='0.16'/>
+    <xacro:property name='chss_h' value='0.08'/>
+    <xacro:property name='chss_mass' value='2'/>
+    <xacro:property name='wheel_to_origin' value='0.07'/>
+    <xacro:property name='wheel_rad' value='0.035'/>
+    <xacro:property name='wheel_wid' value='0.02'/>
+    <xacro:property name='wheel_mass' value='0.05'/>
+    <xacro:property name='caster_rad' value='0.035'/>
     <xacro:property name='caster_mass' value='0.02'/>
     <xacro:property name='front_caster_to_origin' value='0.1'/>
     <xacro:property name='back_caster_to_x' value='0.08'/>
-    <xacro:property name='back_caster_to_y' value='0.06'/> -->
+    <xacro:property name='back_caster_to_y' value='0.06'/>
     <!-- lidar -->
     <xacro:property name='lidar_rad' value='0.035'/>

Commit message: small ad

File: description/constants.xacro (robot description, xacro)
@@ -3,5 +3,5 @@
     <!-- Constants -->
     <!-- REAL ROBOT -->
-    <!-- <xacro:property name='chss_len' value='0.8'/>
+    <xacro:property name='chss_len' value='0.8'/>
     <xacro:property name='chss_wid' value='0.8'/>
     <xacro:property name='chss_h' value='0.325'/>
@@ -15,7 +15,7 @@
     <xacro:property name='front_caster_to_origin' value='0.25'/>
     <xacro:property name='back_caster_to_x' value='0.25'/>
-    <xacro:property name='back_caster_to_y' value='0.25'/> -->
+    <xacro:property name='back_caster_to_y' value='0.25'/>
     <!-- MEJD'S ROBOT -->
-    <xacro:property name='chss_len' value='0.26'/>
+    <!-- <xacro:property name='chss_len' value='0.26'/>
     <xacro:property name='chss_wid' value='0.16'/>
     <xacro:property name='chss_h' value='0.08'/>
@@ -29,5 +29,5 @@
     <xacro:property name='front_caster_to_origin' value='0.1'/>
     <xacro:property name='back_caster_to_x' value='0.08'/>
-    <xacro:property name='back_caster_to_y' value='0.06'/>
+    <xacro:property name='back_caster_to_y' value='0.06'/> -->
     <!-- lidar -->
     <xacro:property name='lidar_rad' value='0.035'/>
