Commit message: getting rid of joint_broad

File: description/robot_core.xacro (robot description, xacro)
@@ -38,5 +38,5 @@
     </link>
     <!-- Right wheel -->
-    <joint name='right_wheel_joint' type='continuous'>
+    <joint name='right_wheel_joint' type='fixed'>
         <parent link='base_link'/>
         <child link='right_wheel'/>
@@ -64,5 +64,5 @@
     </gazebo>
     <!-- Left wheel -->
-    <joint name='left_wheel_joint' type='continuous'>
+    <joint name='left_wheel_joint' type='fixed'>
         <parent link='base_link'/>
         <child link='left_wheel'/>
